File: kicad/Multi-paramter Medicals.kicad_sch (KiCad schematic)
At the start: 30 parts, among them IC1 MPXHZ6400AC6T1, J1 SWITCH, J2 AD8232, J3 MAX30102, J4 DS18B20, J5 12V_BMS, J6 12V_MAIN, J7 LM2596_5V, J8 PUMP, J9 SOLENOID, Q1 IRLB8721, Q2 IRLB8721

Commit message: PCB completed
Parts:
- added C3, C4: 100n, Capacitor_THT:C_Disc_D5.0mm_W2.5mm_P5.00mm, symbol Device:C
- added J10: BUZZER, footprint_:JST_B2B-XH-A, symbol B2B-XH-A:B2B-XH-A
- added J11: OLED, footprint_:JST_B7B-XH-A, symbol B7B-XH-A:B7B-XH-A
- added J12: BP_JST, footprint_:JST_B3B-XH-A, symbol B3B-XH-A:B3B-XH-A
- added JP2: GND_JUMPER, PCM_Jumper_AKL:Jumper_P12.70mm_D0.7mm, symbol Jumper:Jumper_2_Bridged
- added JP3, JP5: 3V3_JUMPER, PCM_Jumper_AKL:Jumper_P15.24mm_D0.7mm, symbol Jumper:Jumper_2_Bridged
- added JP4: PUMP_JUMPER, PCM_Jumper_AKL:Jumper_P15.24mm_D0.7mm, symbol Jumper:Jumper_2_Bridged
- added JP6: 5V_JUMPER, PCM_Jumper_AKL:Jumper_P20.32mm_D0.7mm, symbol Jumper:Jumper_2_Bridged
- added NT1, NT2, NT3, NT4: GND_NetTIE, PCM_Jumper_AKL:Jumper_P7.62mm_D0.7mm, symbol Device:NetTie_2
- added Q3: BC337, Package_TO_SOT_THT:TO-92_Inline_Wide, symbol PCM_Transistor_BJT_AKL:BC337
- added R11: 1k, Resistor_THT:R_Axial_DIN0309_L9.0mm_D3.2mm_P12.70mm_Horizontal, symbol PCM_Elektuur:R
- A1: value ESP32_DevKit_V1_DOIT_30GPIOs -> ESP32_DevKit_V1
- C1: footprint (none) -> Capacitor_THT:C_Disc_D5.0mm_W2.5mm_P5.00mm
- C2: footprint (none) -> Capacitor_THT:CP_Radial_D10.0mm_P7.50mm
- D1, D2: footprint PCM_Diode_THT_AKL:D_DO-41_SOD81_P7.62mm_Horizontal -> Diode_THT:D_DO-41_SOD81_P10.16mm_Horizontal
- D5: value SOLENOID_LED -> VALVE_LED
- IC1: footprint MPXHZ6400AC6T1 -> footprint_:MPXHZ6400AC6T1
- J1: footprint B2B-XH-A:JST_B2B-XH-A -> footprint_:JST_B2B-XH-A
- J2: footprint B5B-XH-A:JST_B5B-XH-A -> footprint_:JST_B5B-XH-A
- J3: footprint B4B-XH-A:JST_B4B-XH-A -> footprint_:JST_B4B-XH-A
- J4: footprint B3B-XH-A:JST_B3B-XH-A -> footprint_:JST_B3B-XH-A
- J5: value 12V_BMS -> BMS; footprint TB002-500-02BE:CUI_TB002-500-02BE -> footprint_:TB002-500-02BE
- J6, J7, J8: footprint TB002-500-02BE:CUI_TB002-500-02BE -> footprint_:TB002-500-02BE
- J9: value SOLENOID -> VALVE; footprint TB002-500-02BE:CUI_TB002-500-02BE -> footprint_:TB002-500-02BE
- Q1, Q2: footprint PCM_Package_TO_SOT_THT_AKL:TO-220-3_Vertical_GDS -> Package_TO_SOT_THT:TO-220-3_Vertical
- R1, R10, R2, R3, R4, R5, R6, R7, R8, R9: footprint (none) -> Resistor_THT:R_Axial_DIN0309_L9.0mm_D3.2mm_P12.70mm_Horizontal
Connections:
- net 3V3: now also C3.2, C4.1, J10.1, J11.2, JP3.1 (A), JP3.2 (B), JP5.1 (A), JP5.2 (B), NT3.1, NT3.2
- net 5V: now also J12.1, JP6.1 (A), JP6.2 (B)
- net GND: now also C3.1, C4.2, J11.1, J12.2, JP2.1 (A), JP2.2 (B), NT1.1, NT1.2, NT2.1, NT2.2, NT4.1, NT4.2, Q3.3 (E)
- net LO+[32]: now also A1.22 (ADC1_CH4/D32); no longer A1.21 (ADC1_CH4/D32)
- net LO-[33]: now also A1.21 (ADC1_CH4/D32); no longer A1.22 (ADC1_CH4/D32)
- net PUMP[26]: now also JP4.1 (A), JP4.2 (B)
- net VOUT: now reaches IC1.4 (VOUT), R1.1 (+)
- net VOUT: now also J12.3
- net D1[23]: now reaches A1.15 (D23)
- net D1[23]: now also J11.4
- net BUZZER: now reaches A1.23 (DAC1/ADC2_CH8/D25)
- net BUZZER: now also R11.1 (+)
- net RES[16]: now reaches A1.6 (RX2/GPIO16)
- net RES[16]: now also J11.5
- net DC[17]: now reaches A1.7 (TX2/GPIO17)
- net DC[17]: now also J11.6
- net CS[5]: now reaches A1.8 (D5)
- net CS[5]: now also J11.7
- net DO[18]: now reaches A1.9 (D18)
- net DO[18]: now also J11.3
- net SOLENOID[27] renamed VALVE[27]
- net SOLENOID_GND renamed VALVE_GND
- new net: J10.2, Q3.1 (C)
- new net: Q3.2 (B), R11.2 (-)
- no-connect marks 22 -> 16
Other:
- moved on the sheet: C2, D1, D2, J1, J5, J6, J7, J8, J9, Q1, Q2, R3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
